File: source/kareems rp2040.kicad_pcb (KiCad board)
At the start: 2 copper layers, 29 x 57 mm, 38 parts, among them J1 USB_C_Receptacle_USB2.0_14P, J2 Conn_01x20, J3 Conn_01x20, J4 Conn_01x03, SW1 SW_Push, U1 RP2040, U2 W25Q16JVSS, U4 MCP1700x-330xxTT, Y1 12MHz

Commit message: eeee
Parts:
- moved R3-1 6.72 mm to (215.0, 98.0)
- moved R4+1 6.72 mm to (214.0, 98.0)
- moved C10 4.05 mm to (216.5, 98.1), turned to 45 degrees
- moved C2 2.77 mm to (213.1, 96.0), turned to 135 degrees
- moved U2 1.60 mm to (213.8, 91.9)
- moved C17 1.59 mm to (212.5, 96.8), turned to 135 degrees
- moved C4 1.21 mm to (217.9, 98.8), turned to 0 degrees
- moved R6 1.20 mm to (212.3, 88.3)
- moved R7 1.10 mm to (214.7, 88.4)
- moved SW1 1.10 mm to (209.6, 85.7)
- moved C8 0.98 mm to (208.1, 99.6)
- moved C9 0.90 mm to (208.1, 100.6)
- moved C11 0.74 mm to (211.8, 97.5), turned to 135 degrees
- moved C7 0.50 mm to (217.1, 109.0)
- moved C1 0.36 mm to (217.0, 108.0)
- renumbered R3 to R3-1, R4 to R4+1
Routing:
- net GND: track 249.8 -> 194.5 mm, vias 13 -> 14
- net +3.3V: track 129.4 -> 144.4 mm, vias 6 -> 7
- net +1V1: track 26.5 -> 18.6 mm, vias 3 -> 2
- net USBD-: track 25.9 -> 33.7 mm
- net USBD+: track 25.5 -> 33.3 mm
- net Net-(U1-USB_DM): track 8.84 -> 1.63 mm
- net Net-(U1-USB_DP): track 8.67 -> 1.46 mm
- net QSPI_SD0: track 11.8 -> 15.7 mm
- net QSPI_SS: track 16.0 -> 18.8 mm
- net QSPI_SD2: track 8.50 -> 10.5 mm
- net QSPI_SCLK: track 14.9 -> 16.3 mm, vias 0 -> 2
- net QSPI_SD1: track 10.00 -> 11.2 mm
- net RUN: track 28.6 -> 29.5 mm
- net GPIO16: track 14.5 -> 15.3 mm
- net GPIO0: track 38.3 -> 39.1 mm
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Other:
- board text added: "10uf"

Commit message: e
Parts:
- moved C13 29.8 mm to (219.8, 77.5), turned to 135 degrees
- moved C7 9.97 mm to (208.2, 104.5), turned to 180 degrees
- turned Y1 to 180 degrees
Routing:
- net GND: track 194.5 -> 178.7 mm, vias 14 -> 20
- net +3.3V: track 144.4 -> 139.7 mm
- net Net-(C16-Pad1): track 8.65 -> 4.77 mm
- net XIN: track 8.33 -> 7.74 mm
