File: source/kareems rp2040.kicad_sch (KiCad schematic)
At the start: 32 parts, among them J1 USB_C_Receptacle_USB2.0_14P, J2 Conn_01x20, J3 Conn_01x20, J4 Conn_01x03, U1 RP2040, U2 W25Q16JVSS, U4 MCP1700x-330xxTT, Y1 12MHz

Commit message: e
Parts:
- added SW1: SW_Push, Button_Switch_SMD:SW_Push_SPST_NO_Alps_SKRK, symbol Switch:SW_Push
Connections:
- net GND: now also SW1.1
- net at R6.1: now also SW1.2
Changed lines of the file:
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@@
+	)
+	(symbol
+		(lib_id "Switch:SW_Push")
+		(at 21.59 106.68 90)
+		(unit 1)
+		(exclude_from_sim no)
+		(in_bom yes)
+		(on_board yes)
+		(dnp no)
+		(fields_autoplaced yes)
+		(property "Reference" "SW1"
+			(at 22.86 105.4099 90)
+			(effects
+				(font
+					(size 1.27 1.27)
+				)
+				(justify right)
+			)
+		)
+		(property "Value" "SW_Push"
+			(at 22.86 107.9499 90)
+			(effects
+				(font
+					(size 1.27 1.27)
+				)
+				(justify right)
+			)
+		)
+		(property "Footprint" "Button_Switch_SMD:SW_Push_SPST_NO_Alps_SKRK"
+			(at 16.51 106.68 0)
+			(effects
+				(font
+					(size 1.27 1.27)
+				)
+				(hide yes)
+			)
+		)
+		(property "Datasheet" "~"
+			(at 16.51 106.68 0)
+			(effects
+				(font
+					(size 1.27 1.27)
+				)
+				(hide yes)
+			)
+		)
+		(property "Description" "Push button switch, generic, two pins"
+			(at 21.59 106.68 0)
+			(effects
+				(font
+					(size 1.27 1.27)
+				)
+				(hide yes)
+			)
+		)
+		(pin "1"
+		)
+		(pin "2"
+		)
+		(instances
+			(project ""
+				(path "/8b916b3e-ac24-44ed-b9f3-8454b1cf38eb"
+					(reference "SW1")
+					(unit 1)
+				)
+			)
+		)
 	)
 	(symbol

Commit message: eeee
Other:
- moved on the sheet: R3, R4
Changed lines of the file:
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@@
 	)
 	(junction
-		(at 48.26 48.26)
-		(diameter 0)
-		(color 0 0 0 0)
-	)
-	(junction
 		(at 78.74 29.21)
 		(diameter 0)
@@
 	)
 	(junction
-		(at 48.26 43.18)
-		(diameter 0)
-		(color 0 0 0 0)
-	)
-	(junction
 		(at 261.62 107.95)
 		(diameter 0)
@@
 	)
 	(junction
+		(at 48.26 44.45)
+		(diameter 0)
+		(color 0 0 0 0)
+	)
+	(junction
 		(at 127 30.48)
 		(diameter 0)
@@
 	)
 	(junction
+		(at 48.26 48.26)
+		(diameter 0)
+		(color 0 0 0 0)
+	)
+	(junction
 		(at 172.72 30.48)
 		(diameter 0)
@@
 	(wire
 		(pts
+			(xy 116.84 104.14) (xy 118.11 104.14)
+		)
+		(stroke
+			(width 0)
+			(type default)
+		)
+	)
+	(wire
+		(pts
 			(xy 48.26 36.83) (xy 60.96 36.83)
 		)
@@
 	(wire
 		(pts
-			(xy 50.8 43.18) (xy 48.26 43.18)
+			(xy 106.68 111.76) (xy 118.11 111.76)
 		)
 		(stroke
@@
 	(wire
 		(pts
-			(xy 106.68 111.76) (xy 118.11 111.76)
+			(xy 106.68 101.6) (xy 109.22 101.6)
 		)
 		(stroke
@@
 	(wire
 		(pts
-			(xy 115.57 101.6) (xy 118.11 101.6)
+			(xy 46.99 104.14) (xy 48.26 104.14)
 		)
 		(stroke
@@
 	(wire
 		(pts
-			(xy 46.99 104.14) (xy 48.26 104.14)
+			(xy 107.95 119.38) (xy 118.11 119.38)
 		)
 		(stroke
@@
 	(wire
 		(pts
-			(xy 107.95 119.38) (xy 118.11 119.38)
+			(xy 262.89 71.12) (xy 262.89 77.47)
 		)
 		(stroke
@@
 	(wire
 		(pts
-			(xy 262.89 71.12) (xy 262.89 77.47)
+			(xy 48.26 48.26) (xy 48.26 49.53)
 		)
 		(stroke
@@
 	(wire
 		(pts
-			(xy 48.26 48.26) (xy 48.26 49.53)
-		)
-		(stroke
-			(width 0)
-			(type default)
-		)
-	)
-	(wire
-		(pts
 			(xy 208.28 120.65) (xy 208.28 129.54)
 		)
@@
 	(wire
 		(pts
-			(xy 115.57 104.14) (xy 118.11 104.14)
-		)
-		(stroke
-			(width 0)
-			(type default)
-		)
-	)
-	(wire
-		(pts
 			(xy 133.35 69.85) (xy 133.35 71.12)
 		)
@@
 	(wire
 		(pts
-			(xy 93.98 104.14) (xy 107.95 104.14)
+			(xy 116.84 101.6) (xy 118.11 101.6)
 		)
 		(stroke
@@
 	(wire
 		(pts
-			(xy 48.26 41.91) (xy 48.26 43.18)
+			(xy 69.85 36.83) (xy 69.85 38.1)
 		)
 		(stroke
@@
 	(wire
 		(pts
-			(xy 69.85 36.83) (xy 69.85 38.1)
+			(xy 149.86 58.42) (xy 161.29 58.42)
 		)
 		(stroke
@@
 	(wire
 		(pts
-			(xy 149.86 58.42) (xy 161.29 58.42)
+			(xy 48.26 48.26) (xy 63.5 48.26)
 		)
 		(stroke
@@
 	(wire
 		(pts
-			(xy 93.98 101.6) (xy 107.95 101.6)
+			(xy 48.26 44.45) (xy 57.15 44.45)
 		)
 		(stroke
@@
 	(wire
 		(pts
-			(xy 50.8 48.26) (xy 48.26 48.26)
+			(xy 208.28 107.95) (xy 210.82 107.95)
 		)
 		(stroke
@@
 	(wire
 		(pts
-			(xy 208.28 107.95) (xy 210.82 107.95)
+			(xy 106.68 104.14) (xy 109.22 104.14)
 		)
 		(stroke
@@
 	(wire
 		(pts
-			(xy 48.26 43.18) (xy 48.26 44.45)
+			(xy 48.26 41.91) (xy 48.26 44.45)
 		)
 		(stroke
@@
 	(global_label "USBD-"
 		(shape bidirectional)
-		(at 50.8 43.18 0)
+		(at 57.15 44.45 0)
 		(fields_autoplaced yes)
 		(effects
@@
 		)
 		(property "Intersheetrefs" "${INTERSHEET_REFS}"
-			(at 61.5489 43.18 0)
+			(at 67.8989 44.45 0)
 			(effects
 				(font
@@
 	(global_label "USBD+"
 		(shape bidirectional)
-		(at 50.8 48.26 0)
+		(at 63.5 48.26 0)
 		(fields_autoplaced yes)
 		(effects
@@
 		)
 		(property "Intersheetrefs" "${INTERSHEET_REFS}"
-			(at 61.5489 48.26 0)
+			(at 74.2489 48.26 0)
 			(effects
 				(font
@@
 	(global_label "USBD+"
 		(shape bidirectional)
-		(at 93.98 104.14 180)
+		(at 106.68 104.14 180)
 		(fields_autoplaced yes)
 		(effects
@@
 		)
 		(property "Intersheetrefs" "${INTERSHEET_REFS}"
-			(at 83.2311 104.14 0)
+			(at 95.9311 104.14 0)
 			(effects
 				(font
@@
 	(global_label "USBD-"
 		(shape bidirectional)
-		(at 93.98 101.6 180)
+		(at 106.68 101.6 180)
 		(fields_autoplaced yes)
 		(effects
@@
 		)
 		(property "Intersheetrefs" "${INTERSHEET_REFS}"
-			(at 83.2311 101.6 0)
+			(at 95.9311 101.6 0)
 			(effects
 				(font
@@
 	(symbol
 		(lib_id "Device:R")
-		(at 111.76 101.6 90)
+		(at 113.03 101.6 90)
 		(unit 1)
 		(exclude_from_sim no)
@@
 		(fields_autoplaced yes)
 		(property "Reference" "R3"
-			(at 111.76 95.25 90)
+			(at 113.03 95.25 90)
 			(effects
 				(font
@@
 		)
 		(property "Value" "27"
-			(at 111.76 97.79 90)
+			(at 113.03 97.79 90)
 			(effects
 				(font
@@
 		)
 		(property "Footprint" "Resistor_SMD:R_0402_1005Metric"
-			(at 111.76 103.378 90)
+			(at 113.03 103.378 90)
 			(effects
 				(font
@@
 		)
 		(property "Datasheet" "~"
-			(at 111.76 101.6 0)
+			(at 113.03 101.6 0)
 			(effects
 				(font
@@
 		)
 		(property "Description" "Resistor"
-			(at 111.76 101.6 0)
+			(at 113.03 101.6 0)
 			(effects
 				(font
@@
 	(symbol
 		(lib_id "Device:R")
-		(at 111.76 104.14 90)
+		(at 113.03 104.14 90)
 		(unit 1)
 		(exclude_from_sim no)
@@
 		(dnp no)
 		(property "Reference" "R4"
-			(at 111.76 107.442 90)
+			(at 113.03 107.442 90)
 			(effects
 				(font
@@
 		)
 		(property "Value" "27"
-			(at 111.76 109.982 90)
+			(at 113.03 109.982 90)
 			(effects
 				(font
@@
 		)
 		(property "Footprint" "Resistor_SMD:R_0402_1005Metric"
-			(at 111.76 105.918 90)
+			(at 113.03 105.918 90)
 			(effects
 				(font
@@
 		)
 		(property "Datasheet" "~"
-			(at 111.76 104.14 0)
+			(at 113.03 104.14 0)
 			(effects
 				(font
@@
 		)
 		(property "Description" "Resistor"
-			(at 111.76 104.14 0)
+			(at 113.03 104.14 0)
 			(effects
 				(font
